File: dcdc/Power.sch (KiCad schematic (older format))
At the start: 0 parts

Commit message: first end
Parts:
- added C13, C17: 220uF, Capacitor_THT:C_Radial_D10.0mm_H12.5mm_P5.00mm, symbol Device:CP_Small
- added C18: 470uF, Capacitor_THT:C_Radial_D10.0mm_H12.5mm_P5.00mm, symbol Device:CP_Small
- added C19: 1000uF, Capacitor_THT:C_Radial_D10.0mm_H12.5mm_P5.00mm, symbol Device:CP_Small
- added C20: 100nF, Capacitor_THT:C_Rect_L7.2mm_W3.5mm_P5.00mm_FKS2_FKP2_MKS2_MKP2, symbol Device:C_Small
- added D3, D4: 1N4148, Diode_THT:D_DO-35_SOD27_P7.62mm_Horizontal, symbol Diode:1N4148
- added D5: D_Schottky_x2_KCom_AKA, ANDY:TO-220-3_pines_separados, symbol Device:D_Schottky_x2_KCom_AKA
- added L1, L2: L_Core_Ferrite, Diode_THT:D_DO-41_SOD81_P10.16mm_Horizontal, symbol Device:L_Core_Ferrite
- added Q10, Q9: BC327, Package_TO_SOT_THT:TO-92L_Wide, symbol Transistor_BJT:BC327
- added Q11, Q12: IRF540N, ANDY:TO-220-3_pines_separados, symbol Transistor_FET:IRF540N
- added R66, R67: 10k, Resistor_THT:R_Axial_DIN0204_L3.6mm_D1.6mm_P7.62mm_Horizontal, symbol Device:R_Small
- added R68, R69: 30R, Resistor_THT:R_Axial_DIN0204_L3.6mm_D1.6mm_P7.62mm_Horizontal, symbol Device:R_Small
- added TR1: TRANSF5, Transformer_THT:Transformer_Toroid_Tapped_Horizontal_D14.0mm_Amidon-T50, symbol Transformer:TRANSF5
Connections:
- new net: C18.1, D5.2 (K), L2.1
- new net: D5.1 (A), TR1.4
- new net: D5.3 (A), TR1.6
- new net: Q12.1 (G), R69.1
- new net: Q12.2 (D), TR1.3
- new net: Q11.1 (G), R68.1
- new net: Q11.2 (D), TR1.1
- new net: D3.1 (K), Q9.3 (E), R68.2
- new net: D4.1 (K), Q10.3 (E), R69.2
- new net +B_POWER: C17.1, L1.2, TR1.2
- new net GND1: C13.2, C17.2, Q10.1 (C), Q11.3 (S), Q12.3 (S), Q9.1 (C), R66.2, R67.2
- new net GND2: C18.2, C19.2, C20.1, TR1.5
- new net OUT_5V: C19.1, C20.2, L2.2
- new net OUT_E_1: D3.2 (A), Q9.2 (B), R66.1
- new net OUT_E_2: D4.2 (A), Q10.2 (B), R67.1
- new net VCC: C13.1, L1.1
