File: dcdc/USBs.sch (KiCad schematic (older format))
At the start: 0 parts

Commit message: first end
Parts:
- added C12: 100nF, Capacitor_THT:C_Rect_L7.2mm_W3.5mm_P5.00mm_FKS2_FKP2_MKS2_MKP2, symbol Device:C_Small
- added J10, J7, J8, J9: USB_A, usb_port:USB_A, symbol Connector:USB_A
- added Q8: BC548, Package_TO_SOT_THT:TO-92L_Wide, symbol Transistor_BJT:BC548
- added R11: 100k, Resistor_SMD:R_0805_2012Metric_Pad1.20x1.40mm_HandSolder, symbol Device:R_Small
- added R21, R42, R43, R44, R45, R47, R48, R55, R56, R57: 4.7k, Resistor_SMD:R_0805_2012Metric_Pad1.20x1.40mm_HandSolder, symbol Device:R_Small
- added R22, R35, R46, R59: 1k, Resistor_SMD:R_0805_2012Metric_Pad1.20x1.40mm_HandSolder, symbol Device:R_Small
- added R23, R36, R49, R60: 1k, Resistor_THT:R_Axial_DIN0207_L6.3mm_D2.5mm_P10.16mm_Horizontal, symbol Device:R_Small
- added R24, R25, R26, R27, R37, R38, R39, R40, R50, R51, R52, R53, R61, R62, R63, R64: R, Resistor_SMD:R_0603_1608Metric_Pad1.05x0.95mm_HandSolder, symbol Device:R_Small
- added R30, R41, R54, R65: 40m, Resistor_SMD:R_2512_6332Metric_Pad1.52x3.35mm_HandSolder, symbol Device:R_Small
- added R31, R58: 220, Resistor_THT:R_Axial_DIN0204_L3.6mm_D1.6mm_P7.62mm_Horizontal, symbol Device:R_Small
- added R32: 5.1k, Resistor_THT:R_Axial_DIN0204_L3.6mm_D1.6mm_P7.62mm_Horizontal, symbol Device:R_Small
- added R34: 4.9k, Resistor_THT:R_Axial_DIN0204_L3.6mm_D1.6mm_P7.62mm_Horizontal, symbol Device:R_Small
- added U2: LM339, Package_DIP:DIP-14_W7.62mm_LongPads, symbol Comparator:LM339
- added U3, U5: PC817, Package_DIP:DIP-4_W7.62mm, symbol Isolator:PC817
- added U4: TL431LP, Package_TO_SOT_THT:TO-92L_Wide, symbol Reference_Voltage:TL431LP
Connections:
- new net: R31.2, U3.1
- new net: C12.2, U3.2, U4.3 (K)
- new net: C12.1, R32.2, R34.1, U4.1 (REF)
- new net: J7.2 (D-), R26.2, R27.1
- new net: J7.3 (D+), R24.2, R25.1
- new net: R58.2, U5.1
- new net: Q8.1 (C), U5.2
- new net: R22.2, U2.4 (-)
- new net: R23.2, U2.5 (+)
- new net: J8.2 (D-), R39.2, R40.1
- new net: J8.3 (D+), R37.2, R38.1
- new net: R35.2, U2.6 (-)
- new net: R36.2, U2.7 (+)
- new net: J9.2 (D-), R52.2, R53.1
- new net: J9.3 (D+), R50.2, R51.1
- new net: R46.2, U2.10 (-)
- new net: R49.2, U2.11 (+)
- new net: J10.2 (D-), R63.2, R64.1
- new net: J10.3 (D+), R61.2, R62.1
- new net: R59.2, U2.8 (-)
- new net: R60.2, U2.9 (+)
- new net: R43.1, R45.1, R48.1, R56.1, R57.1
- new net: Q8.2 (B), R57.2
- new net +5V_REF: U3.4, U5.4
- new net GND2: Q8.3 (E), R21.1, R30.1, R34.2, R41.1, R54.1, R65.1, U2.12 (V-), U4.2 (A)
- new net GND_USB_1: J7.4 (GND), J7.5 (Shield), R23.1, R25.2, R27.2, R30.2
- new net GND_USB_2: J8.4 (GND), J8.5 (Shield), R36.1, R38.2, R40.2, R41.2
- new net GND_USB_3: J9.4 (GND), J9.5 (Shield), R49.1, R51.2, R53.2, R54.2
- new net GND_USB_4: J10.4 (GND), J10.5 (Shield), R60.1, R62.2, R64.2, R65.2
- new net OUT_5V: J10.1 (VBUS), J7.1 (VBUS), J8.1 (VBUS), J9.1 (VBUS), R11.1, R24.1, R26.1, R31.1, R32.1, R37.1, R39.1, R42.2, R44.2, R47.2, R50.1, R52.1, R55.2, R58.1, R61.1, R63.1, U2.3 (V+)
- new net OUT_COMP_1: R42.1, R43.2, U2.2
- new net OUT_COMP_2: R44.1, R45.2, U2.1
- new net OUT_COMP_3: R47.1, R48.2, U2.13
- new net OUT_COMP_4: R55.1, R56.2, U2.14
- new net REF_C: R11.2, R21.2, R22.1, R35.1, R46.1, R59.1
- new net corriente: U5.3
- new net voltaje: U3.3
